File: SkyFax.kicad_sch (KiCad schematic)
At the start: 59 parts, among them J1 RJ11/12, J2 DE9_Receptacle_MountingHoles, J3 Conn_01x02, Q1 Q_NPN_BEC, Q2 Q_PNP_BEC, Q3 Q_NPN_BEC, Q4 Q_NPN_BEC, Q5 Q_NPN_BEC, Q6 Q_NPN_EBC, SW1 SW_DIP_x08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

Commit message: Sent to fab v1.0
Parts:
- BZ1: footprint (none) -> Buzzer_Beeper:Buzzer_12x9.5RM7.6
- J3: footprint (none) -> Connector_PinHeader_2.54mm:PinHeader_1x02_P2.54mm_Vertical
Connections:
- net AOUT: now also SW1.7; no longer SW1.4
- net EECLK: now also SW1.6; no longer SW1.5
- net GND: now also U1.39 (EP)
- net SDI: now also SW1.4; no longer SW1.3
- net nCTS: now also SW1.5; no longer SW1.2
- net nDCD: now also SW1.3; no longer SW1.8
- net nFSYNC: now also SW1.2; no longer SW1.1
- net nINT: now also SW1.1; no longer SW1.6
- net nRI: now also SW1.8; no longer SW1.7
Changed lines of the file:
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@@
   (junction (at 203.835 62.23) (diameter 0) (color 0 0 0 0)
   )
+  (junction (at 50.8 129.54) (diameter 0) (color 0 0 0 0)
+  )
   (junction (at 254.635 59.69) (diameter 0) (color 0 0 0 0)
   )
@@
     (stroke (width 0) (type default))
   )
+  (wire (pts (xy 50.8 129.54) (xy 53.34 129.54))
+    (stroke (width 0) (type default))
+  )
   (wire (pts (xy 235.585 52.07) (xy 236.855 52.07))
     (stroke (width 0) (type default))
@@
     (effects (font (size 1.27 1.27)) (justify right bottom))
   )
-  (label "nCTS" (at 21.59 180.34 180) (fields_autoplaced)
+  (label "nCTS" (at 21.59 187.96 180) (fields_autoplaced)
     (effects (font (size 1.27 1.27)) (justify right bottom))
   )
-  (label "nRI" (at 21.59 193.04 180) (fields_autoplaced)
+  (label "nRI" (at 21.59 195.58 180) (fields_autoplaced)
     (effects (font (size 1.27 1.27)) (justify right bottom))
   )
-  (label "nFSYNC" (at 21.59 177.8 180) (fields_autoplaced)
+  (label "nFSYNC" (at 21.59 180.34 180) (fields_autoplaced)
     (effects (font (size 1.27 1.27)) (justify right bottom))
   )
@@
     (effects (font (size 1.27 1.27)) (justify left bottom))
   )
-  (label "nINT" (at 21.59 190.5 180) (fields_autoplaced)
+  (label "nINT" (at 21.59 177.8 180) (fields_autoplaced)
     (effects (font (size 1.27 1.27)) (justify right bottom))
   )
@@
     (effects (font (size 1.27 1.27)) (justify right bottom))
   )
-  (label "nDCD" (at 21.59 195.58 180) (fields_autoplaced)
+  (label "nDCD" (at 21.59 182.88 180) (fields_autoplaced)
     (effects (font (size 1.27 1.27)) (justify right bottom))
   )
@@
     (effects (font (size 1.27 1.27)) (justify left bottom))
   )
-  (label "EECLK" (at 21.59 187.96 180) (fields_autoplaced)
+  (label "EECLK" (at 21.59 190.5 180) (fields_autoplaced)
     (effects (font (size 1.27 1.27)) (justify right bottom))
   )
-  (label "SDI" (at 21.59 182.88 180) (fields_autoplaced)
+  (label "SDI" (at 21.59 185.42 180) (fields_autoplaced)
     (effects (font (size 1.27 1.27)) (justify right bottom))
   )
@@
     (effects (font (size 1.27 1.27)) (justify right bottom))
   )
-  (label "AOUT" (at 21.59 185.42 180) (fields_autoplaced)
+  (label "AOUT" (at 21.59 193.04 180) (fields_autoplaced)
     (effects (font (size 1.27 1.27)) (justify right bottom))
   )
@@
       (effects (font (size 1.27 1.27)) (justify left) hide)
     )
-    (property "Footprint" "" (at 68.58 129.54 0)
+    (property "Footprint" "Connector_PinHeader_2.54mm:PinHeader_1x02_P2.54mm_Vertical" (at 68.58 129.54 0)
       (effects (font (size 1.27 1.27)) hide)
     )
@@
     (pin "37")
     (pin "38")
+    (pin "39")
     (pin "4")
     (pin "5")
@@
       (effects (font (size 1.27 1.27)) (justify left))
     )
-    (property "Footprint" "" (at 104.14 148.59 90)
+    (property "Footprint" "Buzzer_Beeper:Buzzer_12x9.5RM7.6" (at 104.14 148.59 90)
       (effects (font (size 1.27 1.27)) hide)
     )

Commit message: Version 2.0 Schematics
Parts:
- removed J2: DE9_Receptacle_MountingHoles, Connector_Dsub:DSUB-9_Female_Horizontal_P2.77x2.84mm_EdgePinOffset9.90mm_Housed_MountingHolesOffset11.32mm, symbol Connector:DE9_Receptacle_MountingHoles
- removed J3: Conn_01x02, Connector_PinHeader_2.54mm:PinHeader_1x02_P2.54mm_Vertical, symbol Connector_Generic:Conn_01x02
- removed SW1: SW_DIP_x08, Button_Switch_SMD:SW_DIP_SPSTx08_Slide_6.7x21.88mm_W6.73mm_P2.54mm_LowProfile_JPin, symbol Switch:SW_DIP_x08
- added C11, C12, C17: 0.1uF, Capacitor_SMD:C_0603_1608Metric, symbol Device:C_Small
- added C13, C16: 4.7uF, Capacitor_SMD:C_0402_1005Metric, symbol Device:C_Small
- added D2, D3: LED, LED_SMD:LED_0201_0603Metric, symbol Device:LED
- added FB3, FB4: FerriteBead_Small, Inductor_SMD:L_0805_2012Metric, symbol Device:FerriteBead_Small
- added J2: USB_B_Micro, Connector_USB:USB_Micro-B_Amphenol_10118193-0001LF_Horizontal, symbol Connector:USB_B_Micro
- added JP1, JP2, JP3, JP4, JP5, JP6, JP7, JP8, JP9: Jumper_2_Open, Connector_PinHeader_2.54mm:PinHeader_1x02_P2.54mm_Vertical, symbol Jumper:Jumper_2_Open
- added U4: CP2102N-Axx-xQFN20, Package_DFN_QFN:SiliconLabs_QFN-20-1EP_3x3mm_P0.5mm, symbol Interface_USB:CP2102N-Axx-xQFN20
- R17: value 10k -> 1k; footprint Resistor_SMD:R_0603_1608Metric -> Resistor_SMD:R_0402_1005Metric; DIGIKEY RNCP0603FTD10K0CT-ND -> 311-1.0KJRCT-ND
- R18, R19: value 10k -> 220; footprint Resistor_SMD:R_0603_1608Metric -> Resistor_SMD:R_0402_1005Metric; DIGIKEY RNCP0603FTD10K0CT-ND -> 1292-WR04X2200FTLCT-ND
- R20: value 10k -> 22.1k; footprint Resistor_SMD:R_0603_1608Metric -> Resistor_SMD:R_0402_1005Metric; DIGIKEY RNCP0603FTD10K0CT-ND -> 311-22.1KLRCT-ND
- R21: value 10k -> 47.5k; footprint Resistor_SMD:R_0603_1608Metric -> Resistor_SMD:R_0402_1005Metric; DIGIKEY RNCP0603FTD10K0CT-ND -> 311-47.5KLRCT-ND
- SW2: footprint (none) -> Button_Switch_SMD:SW_Tactile_SPST_NO_Straight_CK_PTS636Sx25SMTRLFS; DIGIKEY (none) -> CKN12322-1-ND
Connections:
- net +3V3: now also R18.1, R19.1, C11.2, C16.2, C17.2, U4.6 (VDD)
- net AOUT: now also JP1.1 (A); no longer R41.2
- net GND: now also C11.1, C12.1, C13.1, C16.1, C17.1, J2.5 (GND), J2.6 (Shield), U4.12 (GND), U4.21 (GND), U4.3 (GND); no longer R17.2, R18.2, R19.2, R20.2
- net RING: now also FB3.2; no longer C8.1, FB1.2
- net RXD: now also JP6.1 (A)
- net SDI: now also JP3.1 (A)
- net TIP: now also FB4.2; no longer C9.1, FB2.2
- net TXD: now also JP5.1 (A)
- net nCTS: now also JP8.1 (A)
- net nDCD: now also R14.1, JP4.1 (A)
- net nFSYNC: now also JP2.1 (A)
- net nRI: now also JP9.1 (A)
- net nRTS: now also JP7.1 (A)
- net C2A: now reaches R13.1, U1.17 (C2A)
- net VBUS: now reaches R17.1
- net VBUS: now also R20.1, C12.2, C13.2, J2.1 (VBUS), U4.7 (VREGIN)
- net C1A: now reaches R12.1, U1.18 (C1A)
- net CLK: now reaches U1.36 (CLKIN_XTAL1), X1.3 (OUT)
- net at R21.1: now also R20.2, U4.8 (VBUS)
- net at R15.1: now also JP2.2 (B)
- net at R16.1: now also JP3.2 (B)
- new net: C9.1, FB2.2, FB4.1
- new net: D2.2 (A), R18.2
- new net: JP9.2 (B), U4.1 (RS485/GPIO.1)
- new net: JP7.2 (B), U4.16 (~{RTS})
- new net: D3.2 (A), R19.2
- new net: D3.1 (K), U4.19 (~{RXT}/GPIO.3)
- new net: JP1.2 (B), R41.2
- new net: JP5.2 (B), U4.18 (TXD)
- new net: D2.1 (K), U4.20 (~{TXT}/GPIO.2)
- new net: JP8.2 (B), U4.15 (~{CTS})
- new net: JP6.2 (B), U4.17 (RXD)
- new net: JP4.2 (B), U4.2 (CLK/GPIO.0)
- new net: R17.2, U4.9 (~{RST})
- new net: C8.1, FB1.2, FB3.1
- new net USB_DM: J2.2 (D-), U4.5 (D-)
- new net USB_DP: J2.3 (D+), U4.4 (D+)
- no-connect marks 19 -> 21
Other:
- moved on the sheet: BZ1, C1, C10, C2, C3, C4, C41, C5, C6, C7, C8, C9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

Commit message: Layout v1.9 (not finished)
Parts:
- removed JP2, JP3, JP4, JP5, JP6, JP7, JP8, JP9: Jumper_2_Open, Connector_PinHeader_2.54mm:PinHeader_1x02_P2.54mm_Vertical, symbol Jumper:Jumper_2_Open
- added J3: Conn_02x06_Odd_Even, Connector_PinHeader_2.54mm:PinHeader_2x06_P2.54mm_Vertical, symbol Connector_Generic:Conn_02x06_Odd_Even
- added J4: Conn_02x02_Odd_Even, Connector_PinHeader_2.54mm:PinHeader_2x02_P2.54mm_Vertical, symbol Connector_Generic:Conn_02x02_Odd_Even
- U4: footprint Package_DFN_QFN:SiliconLabs_QFN-20-1EP_3x3mm_P0.5mm -> Package_DFN_QFN:SiliconLabs_QFN-20-1EP_3x3mm_P0.5mm_EP1.8x1.8mm
Connections:
- net RXD: now also J3.6 (Pin_6)
- net SDI: now also J4.1 (Pin_1)
- net TXD: now also J3.8 (Pin_8)
- net nCTS: now also J3.2 (Pin_2)
- net nDCD: now also J3.10 (Pin_10)
- net nFSYNC: now also J4.3 (Pin_3)
- net nRI: now also J3.12 (Pin_12)
- net nRTS: now also J3.4 (Pin_4)
- net at R15.1: now also J4.2 (Pin_2)
- net at U4.1 (RS485/GPIO.1): now also J3.9 (Pin_9)
- net at U4.16 (~{RTS}): now also J3.3 (Pin_3)
- net at U4.18 (TXD): now also J3.7 (Pin_7)
- net at U4.15 (~{CTS}): now also J3.1 (Pin_1)
- net at U4.17 (RXD): now also J3.5 (Pin_5)
- net at U4.2 (CLK/GPIO.0): now also J3.11 (Pin_11)
- net at R16.1: now also J4.4 (Pin_4)

Commit message: Sent to fab v2.0
Parts:
- added RV1: (no value), Diode_SMD:D_SMB, symbol Device:R
Connections:
- net RING: now also RV1.2
- net TIP: now also RV1.1
- net 1_N: now reaches C2.2, R13.2
- net 1_P: now reaches C1.2, R12.2
- net C1A renamed C1_P
- net C2A renamed C1_N
Other:
- moved on the sheet: R12, R13
Changed lines of the file:
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@@
     (stroke (width 0) (type default))
   )
+  (wire (pts (xy 258.445 47.625) (xy 258.445 52.07))
+    (stroke (width 0) (type default))
+  )
   (wire (pts (xy 180.975 59.69) (xy 187.96 59.69))
     (stroke (width 0) (type default))
@@
     (stroke (width 0) (type default))
   )
-  (polyline (pts (xy 263.525 15.24) (xy 104.14 15.24))
+  (polyline (pts (xy 265.43 15.24) (xy 104.14 15.24))
     (stroke (width 0) (type dash))
   )
@@
     (stroke (width 0) (type default))
   )
+  (wire (pts (xy 258.445 36.83) (xy 258.445 40.005))
+    (stroke (width 0) (type default))
+  )
   (wire (pts (xy 58.42 176.53) (xy 62.23 176.53))
     (stroke (width 0) (type default))
@@
     (stroke (width 0) (type default))
   )
-  (wire (pts (xy 100.965 57.15) (xy 101.6 57.15))
+  (wire (pts (xy 97.155 57.15) (xy 101.6 57.15))
     (stroke (width 0) (type default))
   )
@@
     (stroke (width 0) (type default))
   )
-  (polyline (pts (xy 263.525 99.06) (xy 263.525 15.24))
+  (polyline (pts (xy 265.43 99.06) (xy 265.43 15.24))
     (stroke (width 0) (type dash))
   )
@@
     (stroke (width 0) (type default))
   )
-  (wire (pts (xy 100.965 52.07) (xy 101.6 52.07))
+  (wire (pts (xy 97.155 52.07) (xy 101.6 52.07))
     (stroke (width 0) (type default))
   )
@@
     (stroke (width 0) (type default))
   )
-  (polyline (pts (xy 104.14 99.06) (xy 263.525 99.06))
+  (polyline (pts (xy 104.14 99.06) (xy 265.43 99.06))
     (stroke (width 0) (type dash))
   )
@@
     (effects (font (size 1.27 1.27)) (justify right bottom))
   )
-  (label "C1A" (at 93.345 52.07 180) (fields_autoplaced)
+  (label "C1_P" (at 89.535 52.07 180) (fields_autoplaced)
     (effects (font (size 1.27 1.27)) (justify right bottom))
   )
@@
     (effects (font (size 1.27 1.27)) (justify right bottom))
   )
-  (label "C1A" (at 76.2 59.69 0) (fields_autoplaced)
-    (effects (font (size 1.27 1.27)) (justify left bottom))
-  )
   (label "EECLK" (at 25.4 60.96 180) (fields_autoplaced)
     (effects (font (size 1.27 1.27)) (justify right bottom))
@@
     (effects (font (size 1.27 1.27)) (justify right bottom))
   )
-  (label "EESDO" (at 124.46 148.59 0) (fields_autoplaced)
+  (label "C1_N" (at 76.2 64.77 0) (fields_autoplaced)
     (effects (font (size 1.27 1.27)) (justify left bottom))
   )
-  (label "C2A" (at 76.2 64.77 0) (fields_autoplaced)
+  (label "EESDO" (at 124.46 148.59 0) (fields_autoplaced)
     (effects (font (size 1.27 1.27)) (justify left bottom))
   )
@@
     (effects (font (size 1.27 1.27)) (justify right bottom))
   )
+  (label "1_N" (at 99.695 57.15 270) (fields_autoplaced)
+    (effects (font (size 1.27 1.27)) (justify right bottom))
+  )
   (label "nCTS" (at 25.4 101.6 180) (fields_autoplaced)
     (effects (font (size 1.27 1.27)) (justify right bottom))
   )
+  (label "C1_P" (at 76.2 59.69 0) (fields_autoplaced)
+    (effects (font (size 1.27 1.27)) (justify left bottom))
+  )
   (label "AOUT" (at 25.4 111.76 180) (fields_autoplaced)
     (effects (font (size 1.27 1.27)) (justify right bottom))
@@
     (effects (font (size 1.27 1.27)) (justify right bottom))
   )
+  (label "1_P" (at 99.695 52.07 90) (fields_autoplaced)
+    (effects (font (size 1.27 1.27)) (justify left bottom))
+  )
   (label "nDCD" (at 25.4 88.9 180) (fields_autoplaced)
     (effects (font (size 1.27 1.27)) (justify right bottom))
@@
     (effects (font (size 1.27 1.27)) (justify right bottom))
   )
-  (label "C2A" (at 93.345 57.15 180) (fields_autoplaced)
+  (label "C1_N" (at 89.535 57.15 180) (fields_autoplaced)
     (effects (font (size 1.27 1.27)) (justify right bottom))
   )
@@
     )
   )
-  (symbol (lib_id "Device:R") (at 97.155 57.15 90) (unit 1)
+  (symbol (lib_id "Device:R") (at 93.345 57.15 90) (unit 1)
     (in_bom yes) (on_board yes) (dnp no)
-    (property "Reference" "R13" (at 97.155 54.61 90)
+    (property "Reference" "R13" (at 93.345 54.61 90)
       (effects (font (size 1.27 1.27)))
     )
-    (property "Value" "56.2" (at 97.155 57.15 90)
+    (property "Value" "56.2" (at 93.345 57.15 90)
       (effects (font (size 1.27 1.27)))
     )
-    (property "Footprint" "Resistor_SMD:R_1206_3216Metric" (at 97.155 58.928 90)
+    (property "Footprint" "Resistor_SMD:R_1206_3216Metric" (at 93.345 58.928 90)
       (effects (font (size 1.27 1.27)) hide)
     )
-    (property "Datasheet" "~" (at 97.155 57.15 0)
+    (property "Datasheet" "~" (at 93.345 57.15 0)
       (effects (font (size 1.27 1.27)) hide)
     )
-    (property "DIGIKEY" "RNCP1206FTD56R2CT-ND" (at 97.155 57.15 0)
+    (property "DIGIKEY" "RNCP1206FTD56R2CT-ND" (at 93.345 57.15 0)
       (effects (font (size 1.27 1.27)) hide)
     )
@@
     )
   )
+  (symbol (lib_id "Device:R") (at 258.445 43.815 0) (unit 1)
+    (in_bom yes) (on_board yes) (dnp no) (fields_autoplaced)
+    (property "Reference" "RV1" (at 260.35 42.545 0)
+      (effects (font (size 1.27 1.27)) (justify left))
+    )
+    (property "Value" "" (at 260.35 45.085 0)
+      (effects (font (size 1.27 1.27)) (justify left) hide)
+    )
+    (property "Footprint" "Diode_SMD:D_SMB" (at 256.667 43.815 90)
+      (effects (font (size 1.27 1.27)) hide)
+    )
+    (property "Datasheet" "~" (at 258.445 43.815 0)
+      (effects (font (size 1.27 1.27)) hide)
+    )
+    (property "KICAD" "P3100SALRPTR-ND" (at 258.445 43.815 0)
+      (effects (font (size 1.27 1.27)) hide)
+    )
+    (pin "1")
+    (pin "2")
+    (instances
+      (project "SkyFax"
+        (path "/8648f108-1e45-4954-a197-b251f5522881"
+          (reference "RV1") (unit 1)
+        )
+      )
+    )
+  )
   (symbol (lib_id "SkyFax:SI2494-A-FM") (at 50.8 77.47 0) (unit 1)
     (in_bom yes) (on_board yes) (dnp no)
@@
     )
   )
-  (symbol (lib_id "Device:R") (at 97.155 52.07 90) (unit 1)
+  (symbol (lib_id "Device:R") (at 93.345 52.07 90) (unit 1)
     (in_bom yes) (on_board yes) (dnp no)
-    (property "Reference" "R12" (at 97.155 49.53 90)
+    (property "Reference" "R12" (at 93.345 49.53 90)
       (effects (font (size 1.27 1.27)))
     )
-    (property "Value" "56.2" (at 97.155 52.07 90)
+    (property "Value" "56.2" (at 93.345 52.07 90)
       (effects (font (size 1.27 1.27)))
     )
-    (property "Footprint" "Resistor_SMD:R_1206_3216Metric" (at 97.155 53.848 90)
+    (property "Footprint" "Resistor_SMD:R_1206_3216Metric" (at 93.345 53.848 90)
       (effects (font (size 1.27 1.27)) hide)
     )
-    (property "Datasheet" "~" (at 97.155 52.07 0)
+    (property "Datasheet" "~" (at 93.345 52.07 0)
       (effects (font (size 1.27 1.27)) hide)
     )
-    (property "DIGIKEY" "RNCP1206FTD56R2CT-ND" (at 97.155 52.07 0)
+    (property "DIGIKEY" "RNCP1206FTD56R2CT-ND" (at 93.345 52.07 0)
       (effects (font (size 1.27 1.27)) hide)
     )

Commit message: Schematics v3.0
Parts:
- removed BZ1: Buzzer, Buzzer_Beeper:Buzzer_12x9.5RM7.6, symbol Device:Buzzer
- removed C10: 0.01uF, Capacitor_SMD:C_0603_1608Metric, symbol Device:C_Small
- removed C11, C12, C17, C41, C5, C50, C52, C6: 0.1uF, Capacitor_SMD:C_0603_1608Metric, symbol Device:C_Small
- removed C13, C16: 4.7uF, Capacitor_SMD:C_0402_1005Metric, symbol Device:C_Small
- removed C3: 10nF, Capacitor_SMD:C_0805_2012Metric, symbol Device:C_Small
- removed C4: 1uF, Capacitor_SMD:C_1206_3216Metric, symbol Device:C_Polarized_US
- removed C51: 0.22uF, Capacitor_SMD:C_0603_1608Metric, symbol Device:C_Small
- removed C7: 2.7nF, Capacitor_SMD:C_0603_1608Metric, symbol Device:C_Small
- removed C8, C9: 680pF, Capacitor_SMD:C_1812_4532Metric, symbol Device:C_Small
- removed D1: DF04S, Diode_SMD:Diode_Bridge_OnSemi_SDIP-4L, symbol Diode_Bridge:ABS4
- removed D2, D3: LED, LED_SMD:LED_0201_0603Metric, symbol Device:LED
- removed FB1, FB2, FB3, FB4: FerriteBead_Small, Inductor_SMD:L_0805_2012Metric, symbol Device:FerriteBead_Small
- removed J2: USB_B_Micro, Connector_USB:USB_Micro-B_Amphenol_10118193-0001LF_Horizontal, symbol Connector:USB_B_Micro
- removed J3: Conn_02x06_Odd_Even, Connector_PinHeader_2.54mm:PinHeader_2x06_P2.54mm_Vertical, symbol Connector_Generic:Conn_02x06_Odd_Even
- removed J4: Conn_02x02_Odd_Even, Connector_PinHeader_2.54mm:PinHeader_2x02_P2.54mm_Vertical, symbol Connector_Generic:Conn_02x02_Odd_Even
- removed JP1: Jumper_2_Open, Connector_PinHeader_2.54mm:PinHeader_1x02_P2.54mm_Vertical, symbol Jumper:Jumper_2_Open
- removed Q1, Q4, Q5: Q_NPN_BEC, Package_TO_SOT_SMD:SOT-23, symbol Device:Q_NPN_BEC
- removed Q2: Q_PNP_BEC, Package_TO_SOT_SMD:SOT-23, symbol Device:Q_PNP_BEC
- removed Q3: Q_NPN_BEC, Package_TO_SOT_SMD:SOT-23, symbol Device:Q_NPN_BCE
- removed Q6: Q_NPN_EBC, Package_TO_SOT_THT:TO-92, symbol Device:Q_NPN_EBC
- removed R1: 1.07k, Resistor_SMD:R_2010_5025Metric, symbol Device:R
- removed R10: 536, Resistor_SMD:R_1210_3225Metric, symbol Device:R
- removed R11: 73.2, Resistor_SMD:R_2010_5025Metric, symbol Device:R
- removed R14, R15, R16, R22, R23, R24: 10k, Resistor_SMD:R_0603_1608Metric, symbol Device:R
- removed R17: 1k, Resistor_SMD:R_0402_1005Metric, symbol Device:R
- removed R18, R19: 220, Resistor_SMD:R_0402_1005Metric, symbol Device:R
- removed R2, R41: 150, Resistor_SMD:R_0603_1608Metric, symbol Device:R
- removed R20: 22.1k, Resistor_SMD:R_0402_1005Metric, symbol Device:R
- removed R21: 47.5k, Resistor_SMD:R_0402_1005Metric, symbol Device:R
- removed R3: 3.65k, Resistor_SMD:R_2010_5025Metric, symbol Device:R
- removed R4: 2.49k, Resistor_SMD:R_1206_3216Metric, symbol Device:R
- removed R5, R6: 100k, Resistor_SMD:R_1210_3225Metric, symbol Device:R
- removed R7, R8: 20M, Resistor_SMD:R_2512_6332Metric, symbol Device:R
- removed R9: 1M, Resistor_SMD:R_1206_3216Metric, symbol Device:R
- removed RV1: (no value), Diode_SMD:D_SMB, symbol Device:R
- removed SW2: SW_Push, Button_Switch_SMD:SW_Tactile_SPST_NO_Straight_CK_PTS636Sx25SMTRLFS, symbol Switch:SW_Push
- removed U1: Si2494-A-FM, Package_DFN_QFN:QFN-38-1EP_5x7mm_P0.5mm_EP3.15x5.15mm, symbol SkyFax:SI2494-A-FM
- removed U2: Si3018, Package_SO:SOIC-16_3.9x9.9mm_P1.27mm, symbol SkyFax:SI3018-F-FSR
- removed U3: 25LC640AT-E/SN, Package_SO:SOIC-8_3.9x4.9mm_P1.27mm, symbol Memory_EEPROM:25LCxxx
- removed U4: CP2102N-Axx-xQFN20, Package_DFN_QFN:SiliconLabs_QFN-20-1EP_3x3mm_P0.5mm_EP1.8x1.8mm, symbol Interface_USB:CP2102N-Axx-xQFN20
- removed X1: ECS-2520MV-xxx-xx, Oscillator:Oscillator_SMD_ECS_2520MV-xxx-xx-4Pin_2.5x2.0mm, symbol Oscillator:ECS-2520MV-xxx-xx
- removed Z1: D_Zener, Diode_SMD:D_SOD-123, symbol Device:D_Zener
- added J4: Conn_02x08_Odd_Even, Connector_PinSocket_2.54mm:PinSocket_2x08_P2.54mm_Vertical, symbol Connector_Generic:Conn_02x08_Odd_Even
- added J5, J6: Conn_01x02, Connector_PinSocket_2.54mm:PinSocket_1x02_P2.54mm_Vertical, symbol Connector_Generic:Conn_01x02
- C1, C2: footprint Capacitor_SMD:C_1812_4532Metric -> FaxCam:C_1808
Connections:
- net GND: now also J4.15 (Pin_15)
- net SI3018/C1A: now reaches C1.1
- net SI3018/C1A: now also J5.1 (Pin_1)
- net SI3018/C2A: now reaches C2.1
- net SI3018/C2A: now also J5.2 (Pin_2)
- net 1_N: no longer names the net of C2.2, R13.2
- net 1_P: no longer names the net of C1.2, R12.2
- net C1_N renamed SI2494/C2A
- net C1_P renamed SI2494/C1A
- net RING renamed SI3018/RING
- net SI3018/RING: now also J6.2 (Pin_2)
- net TIP renamed SI3018/TIP
- net SI3018/TIP: now also J6.1 (Pin_1)
- new net SI2494/3V3: J4.1 (Pin_1)
- new net SI2494/CTS: J4.9 (Pin_9)
- new net SI2494/DCD: J4.13 (Pin_13)
- new net SI2494/RI: J4.11 (Pin_11)
- new net SI2494/RTS: J4.7 (Pin_7)
- new net SI2494/RXD: J4.5 (Pin_5)
- new net SI2494/TXD: J4.3 (Pin_3)
- new net USB_Serial/3V3: J4.2 (Pin_2)
- new net USB_Serial/CTS: J4.10 (Pin_10)
- new net USB_Serial/DCD: J4.14 (Pin_14)
- new net USB_Serial/GND: J4.16 (Pin_16)
- new net USB_Serial/RI: J4.12 (Pin_12)
- new net USB_Serial/RTS: J4.8 (Pin_8)
- new net USB_Serial/RXD: J4.6 (Pin_6)
- new net USB_Serial/TXD: J4.4 (Pin_4)
- no-connect marks 21 -> 4
Other:
- added sheet SI2494 (si2494.kicad_sch)
- added sheet SI3018 (si3018.kicad_sch)
- added sheet USB_Serial (usb_serial.kicad_sch)
- note removed: "https://www.skyworksinc.com/-/media/Skyworks/SL/documents/public/data-sheets/Si2494-39.pdf Page 12 (Typical Application Schematic)"
