File: si3018.kicad_sch (KiCad schematic)
At the start: 32 parts, among them Q1 Q_NPN_BEC, Q2 Q_PNP_BEC, Q3 Q_NPN_BEC, Q4 Q_NPN_BEC, Q5 Q_NPN_BEC, U2 Si3018

Commit message: Sent to fab v3.0
Parts:
- C10: DIGIKEY 2679-C0603X7R160-103MNETR-ND -> 2679-C0603X7R160-103MNE-CT-ND
- C3: DIGIKEY 2679-C0805X7R251-103KNETR-ND -> 2679-C0805X7R251-103KNE-CT-ND
- C4: DIGIKEY PCE3935CT-ND -> PCE3912CT-ND
- C5, C6: DIGIKEY 2679-C0603X7R160-104MNETR-ND -> 2679-C0603X7R160-104MNE-CT-ND
- C7: DIGIKEY 2679-C0603X7R500-272MNETR-ND -> 2679-C0603X7R500-272MNE-CT-ND
Changed lines of the file:
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@@
       (effects (font (size 1.27 1.27)) hide)
     )
-    (property "DIGIKEY" "2679-C0603X7R500-272MNETR-ND" (at 124.46 52.07 0)
+    (property "DIGIKEY" "2679-C0603X7R500-272MNE-CT-ND" (at 124.46 52.07 0)
       (effects (font (size 1.27 1.27)) hide)
     )
@@
       (effects (font (size 1.27 1.27)) hide)
     )
-    (property "DIGIKEY" "2679-C0805X7R251-103KNETR-ND" (at 180.34 73.66 0)
+    (property "DIGIKEY" "2679-C0805X7R251-103KNE-CT-ND" (at 180.34 73.66 0)
       (effects (font (size 1.27 1.27)) hide)
     )
@@
       (effects (font (size 1.27 1.27)) hide)
     )
-    (property "DIGIKEY" "2679-C0603X7R160-104MNETR-ND" (at 69.85 107.95 0)
+    (property "DIGIKEY" "2679-C0603X7R160-104MNE-CT-ND" (at 69.85 107.95 0)
       (effects (font (size 1.27 1.27)) hide)
     )
@@
       (effects (font (size 1.27 1.27)) hide)
     )
-    (property "DIGIKEY" "2679-C0603X7R160-103MNETR-ND" (at 168.275 73.66 0)
+    (property "DIGIKEY" "2679-C0603X7R160-103MNE-CT-ND" (at 168.275 73.66 0)
       (effects (font (size 1.27 1.27)) hide)
     )
@@
       (effects (font (size 1.27 1.27)) hide)
     )
-    (property "DIGIKEY" "PCE3935CT-ND" (at 114.3 60.96 0)
+    (property "DIGIKEY" "PCE3912CT-ND" (at 114.3 60.96 0)
       (effects (font (size 1.27 1.27)) hide)
     )
@@
       (effects (font (size 1.27 1.27)) hide)
     )
-    (property "DIGIKEY" "2679-C0603X7R160-104MNETR-ND" (at 73.66 107.95 0)
-      (effects (font (size 1.27 1.27)) hide)
-    )
+    (property "DIGIKEY" "2679-C0603X7R160-104MNE-CT-ND" (at 73.66 107.95 0)
+      (effects (font (size 1.27 1.27)) hide)
+    )

Commit message: Version 3.0 ERC/DRC fixes
Changed lines of the file:
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@@
+    )
+  )
+  (symbol (lib_id "power:PWR_FLAG") (at 102.87 115.57 0) (unit 1)
+    (in_bom yes) (on_board yes) (dnp no) (fields_autoplaced)
+    (property "Reference" "#FLG01" (at 102.87 113.665 0)
+      (effects (font (size 1.27 1.27)) hide)
+    )
+    (property "Value" "PWR_FLAG" (at 102.87 110.49 0)
+      (effects (font (size 1.27 1.27)) hide)
+    )
+    (property "Footprint" "" (at 102.87 115.57 0)
+      (effects (font (size 1.27 1.27)) hide)
+    )
+    (property "Datasheet" "~" (at 102.87 115.57 0)
+      (effects (font (size 1.27 1.27)) hide)
+    )
+    (pin "1")
+    (instances
+      (project "SkyFax"
+        (path "/8648f108-1e45-4954-a197-b251f5522881/605d23de-e47a-44f3-987a-fb8e050dc2c1"
+          (reference "#FLG01") (unit 1)
+        )
+      )
     )
   )
@@
         )
       )
+    )
+  )
+  (symbol (lib_id "power:GND1") (at 102.87 115.57 0) (unit 1)
+    (in_bom yes) (on_board yes) (dnp no) (fields_autoplaced)
+    (property "Reference" "#PWR05" (at 102.87 121.92 0)
+      (effects (font (size 1.27 1.27)) hide)
+    )
+    (property "Value" "GND1" (at 102.87 120.015 0)
+      (effects (font (size 1.27 1.27)))
+    )
+    (property "Footprint" "" (at 102.87 115.57 0)
+      (effects (font (size 1.27 1.27)) hide)
+    )
+    (property "Datasheet" "" (at 102.87 115.57 0)
+      (effects (font (size 1.27 1.27)) hide)
+    )
+    (pin "1")
+    (instances
+      (project "SkyFax"
+        (path "/8648f108-1e45-4954-a197-b251f5522881"
+          (reference "#PWR05") (unit 1)
+        )
+        (path "/8648f108-1e45-4954-a197-b251f5522881/605d23de-e47a-44f3-987a-fb8e050dc2c1"
+          (reference "#PWR012") (unit 1)
+        )
+      )
